File: hardware/bokaka/microcontroller.kicad_sch (KiCad schematic)
At the start: 11 parts, among them U2 STM32L053R8Tx

Commit message: Adding rest of design and pdf
Parts:
- added R5: R, symbol Device:R
Connections:
- net BUZZ_PWM: now also U2.29 (PB10)
- net I2C_SCL: now also U2.61 (PB8)
- net I2C_SDA: now also U2.59 (PB7)
- net LED_STATUS: now also U2.41 (PA8)
- net SWD_SWCLK: now also U2.49 (PA14)
- net SWD_SWDIO: now also U2.46 (PA13)
- net TAP_DATA: now also U2.14 (PA0)
- net TAP_DETECT: now also U2.15 (PA1)
- net UART_RX: now also U2.17 (PA3)
- net UART_TX: now also U2.16 (PA2)
- net USR_BTN0: now also U2.2 (PC13)
- net USR_BTN1: now also U2.3 (PC14)
- net ~{RESET}: now also R5.1
- net ~{BOOT_SEL}: now reaches U2.60 (BOOT0)
- net +3V0 renamed +3V3
- net +3V3: now also R5.2
- no-connect marks 0 -> 37
Other:
- moved on the sheet: C10, C11, C3, C4, C5, C6, C7, C8, C9, FB1
